File: Schematic/Schematic.kicad_sch (KiCad schematic)
At the start: 56 parts, among them J1 DC 5V Input, Q1 NDP6020P, U1 ATmega328P-P, U10 5161AS, U11 5161AS, U12 5161AS, U13 5161AS, U14 YP-05, U16 DFPlayer, U17 MP1584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

Commit message: corrected a but in modifyIsSetting and modifyAlarmIsSetting, it should correct a bug with setup value goind out of bound
Other:
- company: (none) -> Lidwyn
- title: (none) -> Alarm Clock Full Schematic
Changed lines of the file:
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@@
 	(generator_version "9.0")
 	(paper "A3")
+	(title_block
+		(title "Alarm Clock Full Schematic")
+		(date "2025-12-06")
+		(rev "1")
+		(company "Lidwyn")
+	)
 	(rectangle
 		(start 297.18 181.61)
